File: Breadboard Power Supply.kicad_pcb (KiCad board)
At the start: 4 copper layers, 53.6 x 28.8 mm, 36 parts, among them IC1 AP3012KTR-G1, J1 USB-C, J10 Conn_01x02_Male, J11 Conn_01x02_Male, J4 Conn_02x04_Odd_Even, J5 Conn_02x04_Odd_Even, J8 Conn_01x02_Male, J9 Conn_01x02_Male, U1 LM1117DT-ADJ, U2 LM1117DT-ADJ

Commit message: Update
Routing:
- net GND: track 37.7 -> 35.8 mm, vias 8 -> 7
- net +12V: track 66.0 -> 65.2 mm
Changed lines of the file:
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@@
 		)
 		(fp_text user "${REFERENCE}"
-			(at 0 0.004 0)
+			(at 0 -5.969 180)
+			(unlocked yes)
 			(layer "F.Fab")
 			(effects
 				(font
-					(size 1.27 1.27)
-					(thickness 0.254)
+					(size 1 1)
+					(thickness 0.15)
 				)
 			)
 		)
 		(fp_text user "${REFERENCE}"
-			(at 0 -5.969 180)
-			(unlocked yes)
+			(at 0 0.004 0)
 			(layer "F.Fab")
 			(effects
 				(font
-					(size 1 1)
-					(thickness 0.15)
+					(size 1.27 1.27)
+					(thickness 0.254)
 				)
 			)
@@
 	)
 	(segment
-		(start 117.541 84.963)
-		(end 117.541 84.43)
-		(width 0.75)
-		(layer "F.Cu")
-		(net 1)
-	)
-	(segment
 		(start 153.411 83.693)
 		(end 154.559 83.693)
@@
 	)
 	(segment
-		(start 117.541 84.43)
-		(end 118.491 83.48)
-		(width 0.75)
-		(layer "F.Cu")
-		(net 1)
-	)
-	(segment
 		(start 148.651 83.693)
 		(end 148.651 84.43514)
@@
 	)
 	(via
-		(at 118.491 83.48)
-		(size 0.8)
-		(drill 0.4)
-		(layers "F.Cu" "B.Cu")
-		(net 1)
-	)
-	(via
 		(at 108.585 85.217)
 		(size 0.8)
@@
 		(width 0.75)
 		(layer "F.Cu")
-		(net 11)
-	)
-	(segment
-		(start 119.991 84.413)
-		(end 119.441 84.963)
-		(width 0.75)
-		(layer "F.Cu")

Commit message: Update
Parts:
- C1, D1, R12, R13, R9: moved to B.Cu
- moved C11 8.91 mm to (119.9, 82.9)
- moved R13 2.37 mm to (122.5, 80.9), turned to -90 degrees
- moved C1 1.66 mm to (122.6, 83.4)
- moved D1 1.02 mm to (118.5, 81.7)
Routing:
- net Net-(D1-A2): track 8.98 -> 3.35 mm
- net Net-(IC1-FB): track 5.88 -> 1.22 mm
- net +12V: track 65.2 -> 62.6 mm, vias 2 -> 1
- net GND: track 35.8 -> 34.7 mm

Commit message: Update
Parts:
- moved D1 0.76 mm to (118.5, 80.9)
- moved C1 0.51 mm to (122.5, 82.9), turned to 90 degrees
Routing:
- net GND: track 34.7 -> 33.7 mm
Changed lines of the file:
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@@
 	(footprint "Local-Footprints:SODFL3518X115N"
 		(layer "B.Cu")
-		(at 118.491 81.661 180)
+		(at 118.467 80.899 180)
 		(descr "SOD-123F")
 		(tags "Schottky Diode")
@@
 	(footprint "Capacitor_SMD:C_0402_1005Metric"
 		(layer "B.Cu")
-		(at 122.583 83.439)
+		(at 122.5 82.931 90)
 		(descr "Capacitor SMD 0402 (1005 Metric), square (rectangular) end terminal, IPC_7351 nominal, (Body size source: IPC-SM-782 page 76, https://www.pcb-3d.com/wordpress/wp-content/uploads/ipc-sm-782a_amendment_1_and_2.pdf), generated with kicad-footprint-generator")
 		(tags "capacitor")
 		(property "Reference" "C1"
-			(at -0.028 -0.508 360)
+			(at -0.028 -0.508 90)
 			(layer "B.SilkS")
 			(hide yes)
@@
 		)
 		(property "Value" "0.1uF"
-			(at 0 -1.16 360)
+			(at 0 -1.16 90)
 			(layer "B.Fab")
 			(hide yes)
@@
 		)
 		(property "Footprint" "Capacitor_SMD:C_0402_1005Metric"
-			(at 0 0 180)
+			(at 0 0 -90)
 			(unlocked yes)
 			(layer "B.Fab")
@@
 		)
 		(property "Datasheet" ""
-			(at 0 0 180)
+			(at 0 0 -90)
 			(unlocked yes)
 			(layer "B.Fab")
@@
 		)
 		(property "Description" "Unpolarized capacitor"
-			(at 115.669 -77.089 360)
+			(at 115.669 -77.089 90)
 			(layer "B.Fab")
 			(hide yes)
@@
 		)
 		(property "Digi-Key Part Num" "490-14603-1-ND"
-			(at 0 0 360)
+			(at 0 0 90)
 			(layer "B.Fab")
 			(hide yes)
@@
 		)
 		(property "Manufacturer" ""
-			(at 0 0 360)
+			(at 0 0 90)
 			(layer "B.Fab")
 			(hide yes)
@@
 		)
 		(property "Mfg Part Num" ""
-			(at 0 0 360)
+			(at 0 0 90)
 			(layer "B.Fab")
 			(hide yes)
@@
 		)
 		(fp_line
-			(start -0.91 -0.46)
-			(end 0.91 -0.46)
+			(start 0.91 -0.46)
+			(end 0.91 0.46)
 			(stroke
 				(width 0.05)
@@
 		)
 		(fp_line
-			(start -0.91 0.46)
-			(end -0.91 -0.46)
+			(start -0.91 -0.46)
+			(end 0.91 -0.46)
 			(stroke
 				(width 0.05)
@@
 		)
 		(fp_line
-			(start 0.91 -0.46)
-			(end 0.91 0.46)
+			(start 0.91 0.46)
+			(end -0.91 0.46)
 			(stroke
 				(width 0.05)
@@
 		)
 		(fp_line
-			(start 0.91 0.46)
-			(end -0.91 0.46)
+			(start -0.91 0.46)
+			(end -0.91 -0.46)
 			(stroke
 				(width 0.05)
@@
 		)
 		(fp_line
-			(start -0.5 -0.25)
-			(end 0.5 -0.25)
+			(start 0.5 -0.25)
+			(end 0.5 0.25)
 			(stroke
 				(width 0.1)
@@
 		)
 		(fp_line
-			(start -0.5 0.25)
-			(end -0.5 -0.25)
+			(start -0.5 -0.25)
+			(end 0.5 -0.25)
 			(stroke
 				(width 0.1)
@@
 		)
 		(fp_line
-			(start 0.5 -0.25)
-			(end 0.5 0.25)
+			(start 0.5 0.25)
+			(end -0.5 0.25)
 			(stroke
 				(width 0.1)
@@
 		)
 		(fp_line
-			(start 0.5 0.25)
-			(end -0.5 0.25)
+			(start -0.5 0.25)
+			(end -0.5 -0.25)
 			(stroke
 				(width 0.1)
@@
 		)
 		(fp_text user "${REFERENCE}"
-			(at 0 0 360)
+			(at 0 0 90)
 			(layer "B.Fab")
 			(effects
@@
 		)
 		(pad "1" smd roundrect
-			(at -0.48 0)
+			(at -0.48 0 90)
 			(size 0.56 0.62)
 			(layers "B.Cu" "B.Paste" "B.Mask")
@@
 		)
 		(pad "2" smd roundrect
-			(at 0.48 0)
+			(at 0.48 0 90)
 			(size 0.56 0.62)
 			(layers "B.Cu" "B.Paste" "B.Mask")
@@
 	)
 	(segment
-		(start 122.865 81.774)
+		(start 123.587 81.409)
 		(end 122.5 81.409)
 		(width 0.75)
@@
 	)
 	(segment
-		(start 123.952 81.774)
-		(end 122.865 81.774)
-		(width 0.75)
-		(layer "B.Cu")
-		(net 1)
-	)
-	(segment
-		(start 123.952 82.55)
-		(end 123.063 83.439)
+		(start 122.5 82.451)
+		(end 122.5 81.409)
 		(width 0.75)
 		(layer "B.Cu")
@@
 	(segment
 		(start 123.952 81.774)
-		(end 123.952 82.55)
+		(end 123.587 81.409)
 		(width 0.75)
 		(layer "B.Cu")
@@
 	)
 	(segment
-		(start 122.103 83.439)
-		(end 121.287 83.439)
+		(start 121.285 83.441)
+		(end 122.47 83.441)
 		(width 0.75)
 		(layer "B.Cu")
@@
 		(width 0.75)
 		(layer "B.Cu")
+		(net 11)
+	)
+	(segment
+		(start 122.47 83.441)
+		(end 122.5 83.411)
+		(width 0.75)
+		(layer "B.Cu")

Commit message: Update
Parts:
- C10, L2: moved to B.Cu
- moved L2 2.92 mm to (117.7, 77.9), turned to -90 degrees
- moved C10 1.86 mm to (119.8, 77.9), turned to -90 degrees
- moved IC1 0.58 mm to (118.3, 78.3)
Routing:
- net Net-(IC1-FB): track 1.22 -> 6.88 mm, vias 0 -> 1
- net +12V: track 63.0 -> 67.1 mm
- net Net-(D1-A2): track 3.35 -> 5.18 mm, vias 0 -> 1
- net VBUS: track 16.9 -> 15.3 mm

Commit message: Update
Routing:
- net VBUS: track 15.3 -> 16.7 mm
Changed lines of the file:
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@@
 		)
 		(property "Digi-Key Part Num" "445-15751-1-ND"
-			(at 0 0 360)
+			(at 0 0 0)
 			(layer "B.Fab")
 			(hide yes)
@@
 		)
 		(property "Manufacturer" "TDK"
-			(at 0 0 360)
+			(at 0 0 0)
 			(layer "B.Fab")
 			(hide yes)
@@
 		)
 		(property "Mfg Part Num" "MLZ2012P220WT000"
-			(at 0 0 360)
+			(at 0 0 0)
 			(layer "B.Fab")
 			(hide yes)
@@
 	)
 	(segment
+		(start 120.523 77.343)
+		(end 119.507 77.343)
+		(width 0.75)
+		(layer "F.Cu")
+		(net 13)
+	)
+	(segment
 		(start 150.409 83.693)
 		(end 150.155 83.439)
@@
 	)
 	(segment
+		(start 120.777 77.597)
+		(end 120.523 77.343)
+		(width 0.75)
+		(layer "F.Cu")
+		(net 13)
+	)
+	(segment
 		(start 126.752 80.778)
 		(end 126.619 80.645)
@@
 	)
 	(segment
-		(start 120.147 76.967)
+		(start 119.629 76.835)
 		(end 119.761 76.967)
 		(width 0.75)
@@
 	)
 	(segment
-		(start 119.629 76.835)
-		(end 119.761 76.967)
+		(start 119.761 76.967)
+		(end 120.147 76.967)
 		(width 0.75)
 		(layer "B.Cu")
@@
 	)
 	(segment
-		(start 120.777 77.597)
-		(end 120.147 76.967)
+		(start 120.147 76.967)
+		(end 120.777 77.597)
 		(width 0.75)
 		(layer "B.Cu")

Commit message: Update
Parts:
- C1: moved to F.Cu
- moved C1 1.53 mm to (122.6, 84.5), turned to 0 degrees
Routing:
- net +12V: track 67.1 -> 68.7 mm
- net GND: vias 7 -> 8

Commit message: Update
Parts:
- R13, R9: moved to F.Cu
- moved R13 3.28 mm to (121.3, 77.8), turned to 90 degrees
- moved IC1 1.14 mm to (118.3, 77.2)
- moved R9 1.02 mm to (121.3, 79.9)
- moved L2 0.76 mm to (117.0, 77.9)
Routing:
- net GND: track 33.9 -> 37.3 mm, vias 8 -> 7
- net Net-(D1-A2): track 5.18 -> 7.26 mm
- net Net-(R12-Pad2): track 1.01 -> 2.03 mm, vias 0 -> 1
- net VBUS: track 16.7 -> 15.9 mm
- net Net-(IC1-FB): track 6.88 -> 6.59 mm, vias 1 -> 0

Commit message: Update
Parts:
- moved R13 0.51 mm to (121.3, 77.3)
- moved R3 0.51 mm to (137.0, 78.1)
- moved R9 0.25 mm to (121.3, 79.6)
Routing:
- net Net-(D2-Pad2): track 1.61 -> 2.11 mm
Changed lines of the file:
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@@
 	(footprint "Resistor_SMD:R_0402_1005Metric"
 		(layer "F.Cu")
-		(at 137.033 77.597)
+		(at 137.033 78.105)
 		(descr "Resistor SMD 0402 (1005 Metric), square (rectangular) end terminal, IPC_7351 nominal, (Body size source: IPC-SM-782 page 72, https://www.pcb-3d.com/wordpress/wp-content/uploads/ipc-sm-782a_amendment_1_and_2.pdf), generated with kicad-footprint-generator")
 		(tags "resistor")
@@
 	(footprint "Resistor_SMD:R_0402_1005Metric"
 		(layer "F.Cu")
-		(at 121.285 79.881 90)
+		(at 121.285 79.631 90)
 		(descr "Resistor SMD 0402 (1005 Metric), square (rectangular) end terminal, IPC_7351 nominal, (Body size source: IPC-SM-782 page 72, https://www.pcb-3d.com/wordpress/wp-content/uploads/ipc-sm-782a_amendment_1_and_2.pdf), generated with kicad-footprint-generator")
 		(tags "resistor")
@@
 	(footprint "Resistor_SMD:R_0402_1005Metric"
 		(layer "F.Cu")
-		(at 121.285 77.849 90)
+		(at 121.285 77.341 90)
 		(descr "Resistor SMD 0402 (1005 Metric), square (rectangular) end terminal, IPC_7351 nominal, (Body size source: IPC-SM-782 page 72, https://www.pcb-3d.com/wordpress/wp-content/uploads/ipc-sm-782a_amendment_1_and_2.pdf), generated with kicad-footprint-generator")
 		(tags "resistor")
@@
 			(at 2.159 2.667 0)
 			(layer "F.SilkS")
+			(hide yes)
 			(effects
 				(font
@@
 	)
 	(segment
-		(start 121.285 77.339)
-		(end 123.317 77.339)
-		(width 0.75)
-		(layer "F.Cu")
-		(net 1)
-	)
-	(segment
 		(start 115.885 77.155)
 		(end 114.3 78.74)
@@
 	)
 	(segment
-		(start 123.317 77.339)
-		(end 123.952 77.974)
+		(start 121.285 76.831)
+		(end 122.809 76.831)
 		(width 0.75)
 		(layer "F.Cu")
@@
 	)
 	(segment
+		(start 122.809 76.831)
+		(end 123.952 77.974)
+		(width 0.75)
+		(layer "F.Cu")
+		(net 1)
+	)
+	(segment
 		(start 125.522 81.854)
 		(end 124.032 81.854)
@@
 	)
 	(segment
-		(start 121.285 78.359)
-		(end 121.285 79.371)
+		(start 117.007 78.761859)
+		(end 117.833141 79.588)
 		(width 0.75)
 		(layer "F.Cu")
@@
 	)
 	(segment
-		(start 117.007 79.13)
-		(end 117.007 78.105)
+		(start 121.285 77.851)
+		(end 121.285 79.121)
 		(width 0.75)
 		(layer "F.Cu")
@@
 	)
 	(segment
-		(start 118.857859 79.371)
-		(end 118.640859 79.588)
+		(start 120.777 79.121)
+		(end 121.285 79.121)
 		(width 0.75)
 		(layer "F.Cu")
@@
 	)
 	(segment
-		(start 118.640859 79.588)
-		(end 117.465 79.588)
+		(start 117.833141 79.588)
+		(end 120.31 79.588)
 		(width 0.75)
 		(layer "F.Cu")
@@
 	)
 	(segment
-		(start 121.285 79.371)
-		(end 118.857859 79.371)
+		(start 120.31 79.588)
+		(end 120.777 79.121)
 		(width 0.75)
 		(layer "F.Cu")
@@
 	)
 	(segment
-		(start 117.465 79.588)
-		(end 117.007 79.13)
+		(start 117.007 78.105)
+		(end 117.007 78.761859)
 		(width 0.75)
 		(layer "F.Cu")
@@
 	)
 	(segment
-		(start 136.523 77.597)
-		(end 135.763 77.597)
-		(width 0.25)
-		(layer "F.Cu")
-		(net 13)
-	)
-	(segment
 		(start 119.507 78.105)
 		(end 118.237 76.835)
@@
 	)
 	(segment
+		(start 136.523 78.105)
+		(end 135.763 78.105)
+		(width 0.25)
+		(layer "F.Cu")
+		(net 13)
+	)
+	(segment
 		(start 150.409 83.693)
 		(end 150.155 83.439)
@@
 	)
 	(via
-		(at 135.763 77.597)
+		(at 129.921 80.645)
 		(size 0.8)
 		(drill 0.4)
@@
 	)
 	(via
-		(at 129.921 80.645)
+		(at 144.907 81.153)
 		(size 0.8)
 		(drill 0.4)
@@
 	)
 	(via
-		(at 144.907 81.153)
+		(at 150.155 83.439)
 		(size 0.8)
 		(drill 0.4)
@@
 	)
 	(via
-		(at 150.155 83.439)
+		(at 112.649 83.947)
 		(size 0.8)
 		(drill 0.4)
@@
 	)
 	(via
-		(at 112.649 83.947)
+		(at 118.237 76.835)
 		(size 0.8)
 		(drill 0.4)
@@
 	)
 	(via
-		(at 118.237 76.835)
+		(at 135.763 78.105)
 		(size 0.8)
 		(drill 0.4)
@@
 	)
 	(segment
-		(start 121.285 80.391)
+		(start 121.285 80.141)
 		(end 121.285 81.407)
 		(width 0.75)
@@
 	)
 	(segment
-		(start 137.8205 77.3195)
-		(end 137.543 77.597)
+		(start 137.8205 77.8275)
+		(end 137.543 78.105)
 		(width 0.25)
 		(layer "F.Cu")
@@
 	(segment
 		(start 137.8205 76.105)
-		(end 137.8205 77.3195)
+		(end 137.8205 77.8275)
 		(width 0.25)
 		(layer "F.Cu")
